Commit message: Fixed LIDAR sensor URDF to preserve scan topic and namespace

File: robot/description/lidar_sensor.xacro (robot description, xacro)
@@ -1,67 +1,69 @@
 <?xml version="1.0"?>
 <robot xmlns:xacro="http://www.ros.org/wiki/xacro">
-  <!-- Define the Gazebo/Black material -->
-  <material name="Gazebo/Black">
-    <color rgba="0 0 0 1"/>
-  </material>
-  <!-- LIDAR SENSOR JOINT -->
-  <joint name="laser_joint" type="fixed">
-    <parent link="chassis"/>
-    <child link="laser_frame"/>
-    <origin xyz="0.122 0 0.212" rpy="0 0 0"/>
-  </joint>
-  <link name="laser_frame">
-    <visual>
-      <geometry>
-        <cylinder radius="0.05" length="0.04"/>
-      </geometry>
-      <material name="Gazebo/Black"/>
-    </visual>
-    <visual>
-      <origin xyz="0 0 -0.05"/>
-      <geometry>
-        <cylinder radius="0.01" length="0.1"/>
-      </geometry>
-      <material name="Gazebo/Black"/>
-    </visual>
-    <collision>
-      <geometry>
-        <cylinder radius="0.05" length="0.04"/>
-      </geometry>
-    </collision>
-    <!-- Define inertial properties -->
-    <xacro:inertial_cylinder mass="0.1" length="0.04" radius="0.05">
-      <origin xyz="0 0 0" rpy="0 0 0"/>
-    </xacro:inertial_cylinder>
-  </link>
-  <!-- Gazebo sensor and plugin configuration -->
-  <gazebo reference="laser_frame">
-    <material>Gazebo/Black</material>
-    <sensor name="lidar_sensor" type="ray">
-      <pose> 0 0 0 0 0 0 </pose>
-      <visualize>true</visualize>
-      <update_rate>40</update_rate>
-      <ray>
-        <scan>
-          <horizontal>
-            <samples>360</samples>
-            <min_angle>-3.14</min_angle>
-            <max_angle>3.14</max_angle>
-          </horizontal>
-        </scan>
-        <range>
-          <min>0.3</min>
-          <max>12</max>
-          <resolution>0.2</resolution>
-        </range>
-      </ray>
-      <plugin name="laser_controller" filename="libgazebo_ros_ray_sensor.so">
-        <ros>
-          <remap from="out" to="scan"/>
-        </ros>
-        <output_type>sensor_msgs/LaserScan</output_type>
-        <frame_name>laser_frame</frame_name>
-      </plugin>
-    </sensor>
-  </gazebo>
+    <!-- LIDAR SENSOR JOINT -->
+    <joint name="laser_joint" type="fixed">
+        <parent link="chassis"/>
+        <child link="laser_frame"/>
+        <origin xyz="0.122 0 0.212" rpy="0 0 0"/>
+    </joint>
+    <!-- LIDAR SENSOR LINK -->
+    <link name="laser_frame">
+        <visual>
+            <geometry>
+                <cylinder radius="0.05" length="0.04"/>
+            </geometry>
+            <material name="black"/>
+        </visual>
+        <visual>
+            <origin xyz="0 0 -0.05"/>
+            <geometry>
+                <cylinder radius="0.01" length="0.1"/>
+            </geometry>
+            <material name="black"/>
+        </visual>
+        <collision>
+            <geometry>
+                <cylinder radius="0.05" length="0.04"/>
+            </geometry>
+        </collision>
+        <!-- Inertial properties -->
+        <xacro:inertial_cylinder mass="0.1" length="0.04" radius="0.05">
+            <origin xyz="0 0 0" rpy="0 0 0"/>
+        </xacro:inertial_cylinder>
+    </link>
+    <!-- Gazebo settings -->
+    <gazebo reference="laser_frame">
+        <material>Gazebo/Blue</material> <!-- Use only one material -->
+    </gazebo>
+    <!-- LIDAR SENSOR CONFIGURATION -->
+    <gazebo reference="laser_frame">
+        <sensor name="lidar_sensor" type="ray">
+            <pose>0 0 0 0 0 0</pose>
+            <visualize>true</visualize>
+            <update_rate>40</update_rate>
+            <ray>
+                <scan>
+                    <horizontal>
+                        <samples>360</samples>
+                        <min_angle>-3.14</min_angle>
+                        <max_angle>3.14</max_angle>
+                    </horizontal>
+                </scan>
+                <range>
+                    <min>0.3</min>
+                    <max>12</max>
+                    <resolution>0.2</resolution>
+                </range>
+            </ray>
+            <!-- Updated plugin for ROS 2 -->
+            <plugin name="laser_controller" filename="libgazebo_ros_ray_sensor.so">
+                <ros>
+                    <!-- Fixed remapping syntax -->
+                    <argument>~/out:=scan</argument>
+                </ros>
+                <output_type>sensor_msgs/LaserScan</output_type>
+                <frame_name>laser_frame</frame_name>
+            </plugin>
+        </sensor>
+    </gazebo>
 </robot>
